Commit message: revise xacro error in build of humble

File: aip_xx1_description/urdf/sensor_kit.xacro (robot description, xacro)
@@ -20,5 +20,5 @@
     </link>
     <!-- sensor -->
-    <xacro:property name="calibration" value="${load_yaml('$(arg config_dir)/sensor_kit_calibration.yaml')}"/>
+    <xacro:property name="calibration" value="${xacro.load_yaml('$(arg config_dir)/sensor_kit_calibration.yaml')}"/>
     <!-- lidar -->
     <xacro:VLS-128

File: aip_xx1_description/urdf/sensors.xacro (robot description, xacro)
@@ -2,5 +2,5 @@
 <robot name="vehicle" xmlns:xacro="http://ros.org/wiki/xacro">
   <xacro:arg name="config_dir" default="$(find aip_xx1_description)/config"/>
-  <xacro:property name="calibration" value="${load_yaml('$(arg config_dir)/sensors_calibration.yaml')}"/>
+  <xacro:property name="calibration" value="${xacro.load_yaml('$(arg config_dir)/sensors_calibration.yaml')}"/>
   <!-- sensor kit -->
   <xacro:include filename="sensor_kit.xacro"/>
